Commit message: diffbot params in control.yaml

File: jackal_description/urdf/jackal.urdf.xacro (robot description, xacro)
@@ -235,5 +235,5 @@
       </xacro:unless>
     </hardware>
-    <joint name="front_left_wheel_joint">
+    <joint name="front_left_wheel_joint"> <!-- should it be joint name="$(arg prefix)front_left_wheel_joint" -->
       <command_interface name="velocity"/>
       <state_interface name="position"/>

Commit message: $(arg prefix) added to joint names for jackal

File: jackal_description/urdf/jackal.urdf.xacro (robot description, xacro)
@@ -235,20 +235,20 @@
       </xacro:unless>
     </hardware>
-    <joint name="front_left_wheel_joint"> <!-- should it be joint name="$(arg prefix)front_left_wheel_joint" -->
-      <command_interface name="velocity"/>
-      <state_interface name="position"/>
-      <state_interface name="velocity"/>
-    </joint>
-    <joint name="rear_left_wheel_joint">
-      <command_interface name="velocity"/>
-      <state_interface name="position"/>
-      <state_interface name="velocity"/>
-    </joint>
-    <joint name="front_right_wheel_joint">
-      <command_interface name="velocity"/>
-      <state_interface name="position"/>
-      <state_interface name="velocity"/>
-    </joint>
-    <joint name="rear_right_wheel_joint">
+    <joint name="$(arg prefix)front_left_wheel_joint"> <!-- should it be joint name="$(arg prefix)front_left_wheel_joint" -->
+      <command_interface name="velocity"/>
+      <state_interface name="position"/>
+      <state_interface name="velocity"/>
+    </joint>
+    <joint name="$(arg prefix)rear_left_wheel_joint">
+      <command_interface name="velocity"/>
+      <state_interface name="position"/>
+      <state_interface name="velocity"/>
+    </joint>
+    <joint name="$(arg prefix)front_right_wheel_joint">
+      <command_interface name="velocity"/>
+      <state_interface name="position"/>
+      <state_interface name="velocity"/>
+    </joint>
+    <joint name="$(arg prefix)rear_right_wheel_joint">
       <command_interface name="velocity"/>
       <state_interface name="position"/>

Commit message: removed arg prefix from wheel names

File: jackal_description/urdf/jackal.urdf.xacro (robot description, xacro)
@@ -107,5 +107,5 @@
       <origin xyz="0.012  0.002 0.067" rpy="0 0 0"/>
       <mass value="16.523"/>
-      <!-- Moments of inertia ( chassis without wheels ) -->
+      <!-- Moments of inertia: ( chassis without wheels ) -->
       <inertia
         ixx="0.3136" ixy="-0.0008" ixz="0.0164"
@@ -176,5 +176,5 @@
     <child link="rear_fender_link" />
   </joint>
-  <!-- TODO Make this internal_imu_link or something, and use a mixed-in xacro
+  <!-- TODO: Make this internal_imu_link or something, and use a mixed-in xacro
        to supply the joint between it and imu_link. This is important so that imu_link
        always points to the "active" IMU. When an upgrade IMU is connected, the
@@ -191,5 +191,5 @@
     <child link="imu_link" />
   </joint>
-  <!-- TODO Same note as applies to imu_link -->
+  <!-- TODO: Same note as applies to imu_link -->
   <link name="navsat_link">
     <visual>
@@ -235,20 +235,20 @@
       </xacro:unless>
     </hardware>
-    <joint name="$(arg prefix)front_left_wheel_joint"> <!-- should it be joint name="$(arg prefix)front_left_wheel_joint" -->
-      <command_interface name="velocity"/>
-      <state_interface name="position"/>
-      <state_interface name="velocity"/>
-    </joint>
-    <joint name="$(arg prefix)rear_left_wheel_joint">
-      <command_interface name="velocity"/>
-      <state_interface name="position"/>
-      <state_interface name="velocity"/>
-    </joint>
-    <joint name="$(arg prefix)front_right_wheel_joint">
-      <command_interface name="velocity"/>
-      <state_interface name="position"/>
-      <state_interface name="velocity"/>
-    </joint>
-    <joint name="$(arg prefix)rear_right_wheel_joint">
+    <joint name="front_left_wheel_joint"> <!-- should it be joint name="$(arg prefix)front_left_wheel_joint" -->
+      <command_interface name="velocity"/>
+      <state_interface name="position"/>
+      <state_interface name="velocity"/>
+    </joint>
+    <joint name="rear_left_wheel_joint">
+      <command_interface name="velocity"/>
+      <state_interface name="position"/>
+      <state_interface name="velocity"/>
+    </joint>
+    <joint name="front_right_wheel_joint">
+      <command_interface name="velocity"/>
+      <state_interface name="position"/>
+      <state_interface name="velocity"/>
+    </joint>
+    <joint name="rear_right_wheel_joint">
       <command_interface name="velocity"/>
       <state_interface name="position"/>
